Commit message: coloring material

File: urdf/udacity_bot.xacro (robot description, xacro)
@@ -141,7 +141,4 @@
                 <box size="0.05 0.05 0.05"/>
             </geometry>
-            <material name="">
-                <color rgba="1 0 0 1"/>
-            </material>
         </visual>
     </link>
